File: cad/kicad/modbus_relay/modbus_relay.kicad_sch (KiCad schematic)
At the start: 52 parts, among them J10 Conn_02x03_Odd_Even, K1 Relay_SPDT, Q1 BSS138, SW1 SW_Push, U1 LT1785AxS8, U2 ATtiny3227-M

Commit message: Update of kicad and project files
Parts:
- added Q5: BSS138, Package_TO_SOT_SMD:SOT-23, symbol Transistor_FET:IRLML0030
- added R23: 22, Resistor_SMD:R_1206_3216Metric_Pad1.30x1.75mm_HandSolder, symbol Device:R
- added R42: 10k, Resistor_SMD:R_1206_3216Metric_Pad1.30x1.75mm_HandSolder, symbol Device:R
Connections:
- net GND: now also Q5.2 (S); no longer R5.2
- net VCC: now also D5.2 (A), R42.1
- net ES_CMD renamed ~{ESTOP}
- net LED_FAULT renamed ~{LED_FAULT}
- net ~{LED_FAULT}: now also R23.1; no longer D5.2 (A)
- new net: Q5.1 (G), R23.2, R42.2
- new net: Q5.3 (D), R5.2
Other:
- moved on the sheet: D1, D2, D3, D4, D5, D6, D7, D8, D9, H1, H2, H5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

Commit message: Double sided version
Parts:
- removed D7: G, LED_THT:LED_D3.0mm, symbol Device:LED
- removed H1: MountingHole_Pad, MountingHole:MountingHole_3.2mm_M3_DIN965_Pad_TopBottom, symbol Mechanical:MountingHole_Pad
- removed H5: MountingHole, MountingHole:MountingHole_3.2mm_M3, symbol Mechanical:MountingHole
- removed R7: 680, Resistor_SMD:R_1206_3216Metric_Pad1.30x1.75mm_HandSolder, symbol Device:R
- removed TP1, TP2: TestPoint, TestPoint:TestPoint_Loop_D3.50mm_Drill0.9mm_Beaded, symbol Connector:TestPoint
- removed TP10, TP11, TP12, TP13, TP19, TP21, TP22, TP3, TP6: TestPoint_Small, TestPoint:TestPoint_Pad_D1.5mm, symbol Connector:TestPoint_Small
- added R46, R47, R48, R49, R50: 332, Resistor_SMD:R_0805_2012Metric_Pad1.20x1.40mm_HandSolder, symbol Device:R
- added TP1: TestPoint_Probe, TestPoint:TestPoint_Pad_D1.5mm, symbol Connector:TestPoint_Probe
- C1, C31, C4: footprint Capacitor_SMD:C_0603_1608Metric_Pad1.08x0.95mm_HandSolder -> Capacitor_SMD:C_0805_2012Metric_Pad1.18x1.45mm_HandSolder
- FB4, FB5: footprint Inductor_SMD:L_0603_1608Metric -> Inductor_SMD:L_0805_2012Metric
- R1, R11, R2, R23, R3, R39, R4, R40, R41, R42, R43, R44, R5, R6, R8: footprint Resistor_SMD:R_1206_3216Metric_Pad1.30x1.75mm_HandSolder -> Resistor_SMD:R_0805_2012Metric_Pad1.20x1.40mm_HandSolder
- R12: footprint Resistor_SMD:R_0603_1608Metric_Pad0.98x0.95mm_HandSolder -> Resistor_SMD:R_0805_2012Metric_Pad1.20x1.40mm_HandSolder
Connections:
- net GND: now also D1.1 (K), D2.1 (K), D3.1 (K), D4.1 (K), D6.1 (K), D8.1 (K); no longer R1.2, R2.2, R3.2, R4.2, R6.2, R8.2
- net LED_MAINS: now also R4.1; no longer D4.2 (A)
- net LED_RELAY_1: now also R1.1; no longer D1.2 (A)
- net LED_RELAY_2: now also R2.1; no longer D2.2 (A)
- net LED_RELAY_3: now also R3.1; no longer D3.2 (A)
- net LED_RX: now also R6.1; no longer D6.2 (A)
- net RELAY_CHECK_1: now also R47.2; no longer U2.20 (PC3)
- net RELAY_CHECK_2: now also R48.2; no longer U2.21 (PC4)
- net RELAY_CHECK_3: now also R49.2; no longer U2.22 (PC5)
- net VCC: now also R8.1; no longer D8.2 (A)
- net FILT-: now reaches D19.2 (A2), FB4.2, U1.6 (A)
- net at R39.1, U1.2 (~{RE}), U1.3 (DE): now also R50.1; no longer U2.5 (PA4)
- net FILT+: now reaches D19.1 (A1), FB5.2, U1.7 (B)
- net LED_TX: no longer names the net of U2.8 (PA7)
- net LED_TX: now also R46.2
- new net: D4.2 (A), R4.2
- new net: R47.1, U2.20 (PC3)
- new net: R46.1, TP1.1
- new net: D2.2 (A), R2.2
- new net: D3.2 (A), R3.2
- new net: R50.2, U2.5 (PA4)
- new net: D8.2 (A), R8.2
- new net: D6.2 (A), R6.2
- new net: R48.1, U2.21 (PC4)
- new net: R49.1, U2.22 (PC5)
- new net: D1.2 (A), R1.2
Other:
- moved on the sheet: R1, R11, R12, R2, R3, R4, R40, R5, R6, R8
